File: PCB_Option_Maker/PCB_Module_Payement/Modules_pcb_caisse.kicad_sch (KiCad schematic)
At the start: 12 parts, among them J3 Conn_01x08, J4 Conn_01x06, J5 Conn_01x08, J6 Conn_01x04

Commit message: update schematci
Parts:
- added C13, C17, C19: 1u, Capacitor_SMD:C_0402_1005Metric, symbol Device:C_Small
Connections:
- net +5V: now also C13.1, C17.1, C19.1
- net GND: now also C13.2, C17.2, C19.2
Other:
- moved on the sheet: J6
