File: PCB_Option_Maker/PCB_Module_Payement/Modules_pcb_caisse.kicad_sch (KiCad schematic)
At the start: 11 parts, among them J3 Conn_01x08, J4 Conn_01x06, J5 Conn_01x08, J6 Conn_01x04

Commit message: pcb update
Connections:
- net IRQ: now also J3.8 (Pin_8); no longer J3.7 (Pin_7)
- net KEY: now also J4.6 (Pin_6); no longer J4.1 (Pin_1)
- net RSTO: now also J3.2 (Pin_2); no longer J3.8 (Pin_8)
- net SPI1_Miso: now also J3.7 (Pin_7); no longer J3.2 (Pin_2)
- net SPI1_Mosi: now also J3.4 (Pin_4); no longer J3.3 (Pin_3)
- net SS: now also J3.3 (Pin_3); no longer J3.4 (Pin_4)
- net STATE: now also J4.1 (Pin_1); no longer J4.6 (Pin_6)
Changed lines of the file:
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@@
+	(wire
+		(pts
+			(xy 166.37 111.76) (xy 166.37 110.49)
+		)
+		(stroke
+			(width 0)
+			(type default)
+		)
+	)
+	(wire
+		(pts
+			(xy 138.43 102.87) (xy 138.43 101.6)
+		)
+		(stroke
+			(width 0)
+			(type default)
+		)
+	)
+	(wire
+		(pts
+			(xy 138.43 101.6) (xy 139.7 101.6)
+		)
+		(stroke
+			(width 0)
+			(type default)
+		)
+	)
+	(wire
+		(pts
+			(xy 138.43 109.22) (xy 138.43 110.49)
+		)
+		(stroke
+			(width 0)
+			(type default)
+		)
+	)
 	(wire
 		(pts
@@
 	(wire
 		(pts
-			(xy 166.37 111.76) (xy 166.37 110.49)
-		)
-		(stroke
-			(width 0)
-			(type default)
-		)
-	)
-	(wire
-		(pts
-			(xy 138.43 102.87) (xy 138.43 101.6)
-		)
-		(stroke
-			(width 0)
-			(type default)
-		)
-	)
-	(wire
-		(pts
-			(xy 138.43 101.6) (xy 139.7 101.6)
-		)
-		(stroke
-			(width 0)
-			(type default)
-		)
-	)
-	(wire
-		(pts
-			(xy 138.43 109.22) (xy 138.43 110.49)
-		)
-		(stroke
-			(width 0)
-			(type default)
-		)
-	)
-	(wire
-		(pts
 			(xy 138.43 111.76) (xy 138.43 110.49)
 		)
@@
 	(wire
 		(pts
+			(xy 182.88 78.74) (xy 198.12 78.74)
+		)
+		(stroke
+			(width 0)
+			(type default)
+		)
+	)
+	(wire
+		(pts
 			(xy 137.16 100.33) (xy 138.43 100.33)
 		)
@@
 	(wire
 		(pts
-			(xy 182.88 78.74) (xy 198.12 78.74)
-		)
-		(stroke
-			(width 0)
-			(type default)
-		)
-	)
-	(wire
-		(pts
 			(xy 166.37 109.22) (xy 166.37 110.49)
 		)
@@
 		)
 	)
-	(label "RXD"
-		(at 186.69 81.28 180)
+	(label "Bt_TXD"
+		(at 191.77 78.74 180)
 		(effects
 			(font
@@
 		)
 	)
-	(label "TXD"
-		(at 186.69 78.74 180)
+	(label "Bt_RXD"
+		(at 191.77 81.28 180)
 		(effects
 			(font
@@
 		)
 	)
-	(hierarchical_label "SS"
+	(hierarchical_label "Column3"
+		(shape output)
+		(at 165.1 102.87 180)
+		(effects
+			(font
+				(size 1.27 1.27)
+			)
+			(justify right)
+		)
+	)
+	(hierarchical_label "Column1"
+		(shape output)
+		(at 137.16 102.87 180)
+		(effects
+			(font
+				(size 1.27 1.27)
+			)
+			(justify right)
+		)
+	)
+	(hierarchical_label "IRQ"
+		(shape output)
+		(at 102.87 100.33 180)
+		(effects
+			(font
+				(size 1.27 1.27)
+			)
+			(justify right)
+		)
+	)
+	(hierarchical_label "Column4"
+		(shape output)
+		(at 165.1 111.76 180)
+		(effects
+			(font
+				(size 1.27 1.27)
+			)
+			(justify right)
+		)
+	)
+	(hierarchical_label "RSTO"
+		(shape input)
+		(at 102.87 85.09 180)
+		(effects
+			(font
+				(size 1.27 1.27)
+			)
+			(justify right)
+		)
+	)
+	(hierarchical_label "SPI1_Mosi"
 		(shape input)
 		(at 102.87 90.17 180)
-		(effects
-			(font
-				(size 1.27 1.27)
-			)
-			(justify right)
-		)
-	)
-	(hierarchical_label "USART2_RX"
-		(shape output)
-		(at 182.88 78.74 180)
-		(effects
-			(font
-				(size 1.27 1.27)
-			)
-			(justify right)
-		)
-	)
-	(hierarchical_label "KEY"
-		(shape input)
-		(at 198.12 71.12 180)
-		(effects
-			(font
-				(size 1.27 1.27)
-			)
-			(justify right)
-		)
-	)
-	(hierarchical_label "STATE"
-		(shape output)
-		(at 198.12 83.82 180)
-		(effects
-			(font
-				(size 1.27 1.27)
-			)
-			(justify right)
-		)
-	)
-	(hierarchical_label "RSTO"
-		(shape input)
-		(at 102.87 100.33 180)
-		(effects
-			(font
-				(size 1.27 1.27)
-			)
-			(justify right)
-		)
-	)
-	(hierarchical_label "Column3"
-		(shape output)
-		(at 165.1 102.87 180)
-		(effects
-			(font
-				(size 1.27 1.27)
-			)
-			(justify right)
-		)
-	)
-	(hierarchical_label "IRQ"
-		(shape output)
-		(at 102.87 97.79 180)
-		(effects
-			(font
-				(size 1.27 1.27)
-			)
-			(justify right)
-		)
-	)
-	(hierarchical_label "Column1"
-		(shape output)
-		(at 137.16 102.87 180)
-		(effects
-			(font
-				(size 1.27 1.27)
-			)
-			(justify right)
-		)
-	)
-	(hierarchical_label "Column4"
-		(shape output)
-		(at 165.1 111.76 180)
-		(effects
-			(font
-				(size 1.27 1.27)
-			)
-			(justify right)
-		)
-	)
-	(hierarchical_label "SPI1_Mosi"
-		(shape input)
-		(at 102.87 87.63 180)
-		(effects
-			(font
-				(size 1.27 1.27)
-			)
-			(justify right)
-		)
-	)
-	(hierarchical_label "SPI1_Miso"
-		(shape output)
-		(at 102.87 85.09 180)
 		(effects
 			(font
@@
 		)
 	)
+	(hierarchical_label "SS"
+		(shape input)
+		(at 102.87 87.63 180)
+		(effects
+			(font
+				(size 1.27 1.27)
+			)
+			(justify right)
+		)
+	)
 	(hierarchical_label "ROW4"
 		(shape input)
@@
 		)
 	)
+	(hierarchical_label "USART2_RX"
+		(shape output)
+		(at 182.88 78.74 180)
+		(effects
+			(font
+				(size 1.27 1.27)
+			)
+			(justify right)
+		)
+	)
+	(hierarchical_label "ROW2"
+		(shape input)
+		(at 199.39 102.87 180)
+		(effects
+			(font
+				(size 1.27 1.27)
+			)
+			(justify right)
+		)
+	)
+	(hierarchical_label "KEY"
+		(shape input)
+		(at 198.12 83.82 180)
+		(effects
+			(font
+				(size 1.27 1.27)
+			)
+			(justify right)
+		)
+	)
+	(hierarchical_label "STATE"
+		(shape output)
+		(at 198.12 71.12 180)
+		(effects
+			(font
+				(size 1.27 1.27)
+			)
+			(justify right)
+		)
+	)
+	(hierarchical_label "SPI1_Miso"
+		(shape output)
+		(at 102.87 97.79 180)
+		(effects
+			(font
+				(size 1.27 1.27)
+			)
+			(justify right)
+		)
+	)
 	(hierarchical_label "USART2_TX"
 		(shape input)
@@
 		(effects
 			(font
-				(size 1.27 1.27)
-			)
-			(justify right)
-		)
-	)
-	(hierarchical_label "ROW2"
-		(shape input)
-		(at 199.39 102.87 180)
-		(effects
-			(font
