File: PCB_Option_Maker/PCB_Module_Payement/PCB_STM32_Payement.kicad_sch (KiCad schematic)
At the start: 30 parts, among them J8 USB_C_Receptacle_USB2.0, J9 Conn_ST_STDC14, Q1 2N2219, SW1 SW_Push, SW3 SW_Push, U2 STM32G431CBUx, U6 USBLC6-2SC6

Commit message: update schematci
Parts:
- removed C15: 1u, Capacitor_SMD:C_0603_1608Metric, symbol Device:C_Small
- removed C8, C9: C, Capacitor_SMD:C_0402_1005Metric, symbol Device:C_Small
- removed L1: 39n, Inductor_SMD:L_0805_2012Metric, symbol Device:L_Small
- added SW2: SW_Push, Button_Switch_SMD:SW_Push_1P1T_NO_CK_KSC6xxJ, symbol Switch:SW_Push
- C6: value 100n -> 4u7
- R8: footprint (none) -> Resistor_SMD:R_0402_1005Metric
Connections:
- net +3.3V: now also C14.1, U2.21 (VDDA), SW2.2
- net +3.3VA: no longer C14.1, U2.21 (VDDA)
- net +5V: now also BZ1.1 (+); no longer J8.A4 (VBUS), J8.A9 (VBUS), J8.B4 (VBUS), J8.B9 (VBUS), Q1.3 (C), U6.5 (VBUS)
- net BOOT0: now also SW2.1
- net GND: now also Q1.1 (E); no longer BZ1.2 (-)
- net GPIOy_PINy renamed BUZZER
- new net: BZ1.2 (-), Q1.3 (C)
- new net 5V_USB: J8.A4 (VBUS), J8.A9 (VBUS), J8.B4 (VBUS), J8.B9 (VBUS), U6.5 (VBUS)
Other:
- note removed: "Cristal de qwartz ?"
- note removed: "For VDDA"
- moved on the sheet: BZ1, Q1, R6, R8
