File: PCB_Option_Maker/PCB_Module_Payement/PCB_STM32_Payement.kicad_sch (KiCad schematic)
At the start: 30 parts, among them J1 Conn_02x07_Odd_Even, J8 USB_C_Receptacle_USB2.0, J9 Conn_ST_STDC14, Q2 MMBT2222A, SW1 SW_Push, SW2 SW_Push, SW3 SW_Push, U2 STM32G431CBUx, U6 USBLC6-2SC6

Commit message: pcb update
Connections:
- net Column1: now also U2.29 (PC6); no longer U2.28 (PB15)
- net Column2: now also U2.30 (PA8); no longer U2.27 (PB14)
- net Column3: now also U2.31 (PA9); no longer U2.26 (PB13)
- net Column4: now also U2.32 (PA10); no longer U2.25 (PB12)
- net PA7: now also J1.11 (Pin_11); no longer J1.12 (Pin_12)
- net PC13: now also J1.3 (Pin_3); no longer J1.6 (Pin_6)
- net PC14: now also J1.4 (Pin_4); no longer J1.9 (Pin_9)
- net PC15: now also J1.6 (Pin_6); no longer J1.10 (Pin_10)
- net PF0: now also J1.10 (Pin_10); no longer J1.3 (Pin_3)
- net PF1: now also J1.9 (Pin_9); no longer J1.4 (Pin_4)
- net Pb1: now also J1.12 (Pin_12); no longer J1.11 (Pin_11)
- net Row1: now also U2.25 (PB12); no longer U2.32 (PA10)
- net Row2: now also U2.26 (PB13); no longer U2.31 (PA9)
- net Row3: now also U2.27 (PB14); no longer U2.30 (PA8)
- net Row4: now also U2.28 (PB15); no longer U2.29 (PC6)
- net USB_DM renamed USB_D-
- net USB_DP renamed USB_D+
Changed lines of the file:
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@@
 		)
 	)
-	(label "USB_DP"
+	(label "USB_D+"
 		(at 248.92 137.16 180)
 		(effects
@@
 			)
 			(justify right bottom)
-		)
-	)
-	(label "PC15"
-		(at 40.64 60.96 0)
-		(effects
-			(font
-				(size 1.27 1.27)
-			)
-			(justify left bottom)
 		)
 	)
@@
 		)
 	)
-	(label "PC14"
-		(at 27.94 60.96 180)
+	(label "PA7"
+		(at 27.94 63.5 180)
 		(effects
 			(font
@@
 		)
 	)
+	(label "PC15"
+		(at 40.64 55.88 0)
+		(effects
+			(font
+				(size 1.27 1.27)
+			)
+			(justify left bottom)
+		)
+	)
 	(label "NRST"
 		(at 68.58 55.88 0)
@@
 		)
 	)
-	(label "PC13"
-		(at 40.64 55.88 0)
-		(effects
-			(font
-				(size 1.27 1.27)
-			)
-			(justify left bottom)
-		)
-	)
 	(label "USART3_TX"
 		(at 50.8 116.84 0)
@@
 		)
 	)
-	(label "PF0"
-		(at 27.94 53.34 180)
-		(effects
-			(font
-				(size 1.27 1.27)
-			)
-			(justify right bottom)
-		)
-	)
 	(label "SWCLK"
 		(at 278.13 31.75 180)
@@
 		)
 	)
-	(label "USB_DM"
+	(label "USB_D-"
 		(at 269.24 137.16 0)
 		(effects
@@
 		)
 	)
+	(label "PC13"
+		(at 27.94 53.34 180)
+		(effects
+			(font
+				(size 1.27 1.27)
+			)
+			(justify right bottom)
+		)
+	)
 	(label "BUZZER"
 		(at 180.34 91.44 0)
@@
 	)
 	(label "Pb1"
-		(at 27.94 63.5 180)
-		(effects
-			(font
-				(size 1.27 1.27)
-			)
-			(justify right bottom)
-		)
-	)
-	(label "USB_DP"
+		(at 40.64 63.5 0)
+		(effects
+			(font
+				(size 1.27 1.27)
+			)
+			(justify left bottom)
+		)
+	)
+	(label "USB_D+"
 		(at 123.19 81.28 180)
 		(effects
@@
 		)
 	)
+	(label "PC14"
+		(at 40.64 53.34 0)
+		(effects
+			(font
+				(size 1.27 1.27)
+			)
+			(justify left bottom)
+		)
+	)
 	(label "NRST"
 		(at 278.13 26.67 180)
@@
 		)
 	)
-	(label "PF1"
-		(at 40.64 53.34 0)
-		(effects
-			(font
-				(size 1.27 1.27)
-			)
-			(justify left bottom)
-		)
-	)
-	(label "USB_DM"
+	(label "USB_D-"
 		(at 123.19 78.74 180)
 		(effects
@@
 		)
 	)
+	(label "PF0"
+		(at 40.64 60.96 0)
+		(effects
+			(font
+				(size 1.27 1.27)
+			)
+			(justify left bottom)
+		)
+	)
 	(label "SWDIO"
 		(at 128.27 83.82 180)
@@
 		)
 	)
+	(label "PF1"
+		(at 27.94 60.96 180)
+		(effects
+			(font
+				(size 1.27 1.27)
+			)
+			(justify right bottom)
+		)
+	)
 	(label "D-"
 		(at 269.24 132.08 0)
@@
 			)
 			(justify right bottom)
-		)
-	)
-	(label "PA7"
-		(at 40.64 63.5 0)
-		(effects
-			(font
-				(size 1.27 1.27)
-			)
-			(justify left bottom)
 		)
 	)
@@
 		)
 	)
-	(hierarchical_label "Row4"
-		(shape output)
-		(at 71.12 71.12 180)
-		(effects
-			(font
-				(size 1.27 1.27)
-			)
-			(justify right)
-		)
-	)
-	(hierarchical_label "Column2"
-		(shape input)
-		(at 74.93 124.46 180)
-		(effects
-			(font
-				(size 1.27 1.27)
-			)
-			(justify right)
+	(hierarchical_label "Column4"
+		(shape input)
+		(at 115.57 76.2 0)
+		(effects
+			(font
+				(size 1.27 1.27)
+			)
+			(justify left)
 		)
 	)
@@
 			)
 			(justify right)
+		)
+	)
+	(hierarchical_label "Row2"
+		(shape output)
+		(at 74.93 121.92 180)
+		(effects
+			(font
+				(size 1.27 1.27)
+			)
+			(justify right)
+		)
+	)
+	(hierarchical_label "Column3"
+		(shape input)
+		(at 115.57 73.66 0)
+		(effects
+			(font
+				(size 1.27 1.27)
+			)
+			(justify left)
 		)
 	)
@@
 		)
 	)
+	(hierarchical_label "RFID_SS"
+		(shape output)
+		(at 73.66 104.14 180)
+		(effects
+			(font
+				(size 1.27 1.27)
+			)
+			(justify right)
+		)
+	)
+	(hierarchical_label "UART2_TX_Bt"
+		(shape output)
+		(at 123.19 55.88 0)
+		(effects
+			(font
+				(size 1.27 1.27)
+			)
+			(justify left)
+		)
+	)
+	(hierarchical_label "Column2"
+		(shape input)
+		(at 115.57 71.12 0)
+		(effects
+			(font
+				(size 1.27 1.27)
+			)
+			(justify left)
+		)
+	)
+	(hierarchical_label "SPI1_SCK"
+		(shape output)
+		(at 113.03 63.5 0)
+		(effects
+			(font
+				(size 1.27 1.27)
+			)
+			(justify left)
+		)
+	)
+	(hierarchical_label "Column1"
+		(shape input)
+		(at 71.12 71.12 180)
+		(effects
+			(font
+				(size 1.27 1.27)
+			)
+			(justify right)
+		)
+	)
+	(hierarchical_label "Row3"
+		(shape output)
+		(at 74.93 124.46 180)
+		(effects
+			(font
+				(size 1.27 1.27)
+			)
+			(justify right)
+		)
+	)
+	(hierarchical_label "Row4"
+		(shape output)
+		(at 74.93 127 180)
+		(effects
+			(font
+				(size 1.27 1.27)
+			)
+			(justify right)
+		)
+	)
+	(hierarchical_label "UART2_RX_Bt"
+		(shape input)
+		(at 123.19 58.42 0)
+		(effects
+			(font
+				(size 1.27 1.27)
+			)
+			(justify left)
+		)
+	)
 	(hierarchical_label "Row1"
 		(shape output)
-		(at 115.57 76.2 0)
-		(effects
-			(font
-				(size 1.27 1.27)
-			)
-			(justify left)
-		)
-	)
-	(hierarchical_label "RFID_SS"
-		(shape output)
-		(at 73.66 104.14 180)
-		(effects
-			(font
-				(size 1.27 1.27)
-			)
-			(justify right)
-		)
-	)
-	(hierarchical_label "UART2_TX_Bt"
-		(shape output)
-		(at 123.19 55.88 0)
-		(effects
-			(font
-				(size 1.27 1.27)
-			)
-			(justify left)
-		)
-	)
-	(hierarchical_label "SPI1_SCK"
-		(shape output)
-		(at 113.03 63.5 0)
-		(effects
-			(font
-				(size 1.27 1.27)
-			)
-			(justify left)
-		)
-	)
-	(hierarchical_label "UART2_RX_Bt"
-		(shape input)
-		(at 123.19 58.42 0)
-		(effects
-			(font
-				(size 1.27 1.27)
-			)
-			(justify left)
-		)
-	)
-	(hierarchical_label "Column4"
-		(shape input)
 		(at 74.93 119.38 180)
 		(effects
@@
 		)
 	)
-	(hierarchical_label "Column1"
-		(shape input)
-		(at 74.93 127 180)
-		(effects
-			(font
-				(size 1.27 1.27)
-			)
-			(justify right)
-		)
-	)
 	(hierarchical_label "RFID_IRQ"
 		(shape input)
@@
 		)
 	)
-	(hierarchical_label "Column3"
-		(shape input)
-		(at 74.93 121.92 180)
-		(effects
-			(font
-				(size 1.27 1.27)
-			)
-			(justify right)
-		)
-	)
-	(hierarchical_label "Row3"
-		(shape output)
-		(at 115.57 71.12 0)
-		(effects
-			(font
-				(size 1.27 1.27)
-			)
-			(justify left)
-		)
-	)
 	(hierarchical_label "SPI1_Mosi"
 		(shape input)
@@
 		)
 	)
-	(hierarchical_label "Row2"
-		(shape output)
-		(at 115.57 73.66 0)
-		(effects
-			(font
-				(size 1.27 1.27)
-			)
-			(justify left)
-		)
-	)
