File: PCB_Option_Maker/PCB_Module_Payement/untitled.kicad_sch (KiCad schematic)
At the start: 18 parts, among them J7 Conn_01x02, U4 BU33SD5WG-TR

Commit message: update schematci
Parts:
- removed R10: 200, Resistor_SMD:R_0805_1005Metric, symbol Device:R_Small
- added D6, D7: D_Schottky, symbol Device:D_Schottky
- C2, C4, C5: footprint Capacitor_SMD:C_0805_2012Metric -> Capacitor_SMD:C_0402_1005Metric
- R20: value 300 -> 510; footprint Resistor_SMD:R_0805_1005Metric -> Resistor_SMD:R_0402_1005Metric
- R21: footprint Resistor_SMD:R_0805_1005Metric -> Resistor_SMD:R_0402_1005Metric
- R3: value R -> 5k6; footprint (none) -> Resistor_SMD:R_0402_1005Metric
- R4: value 4.99K -> 49k9
- R5: value 1K -> 10k
- U3: MPN (none) -> 171013801
Connections:
- net +3.3V: now also R20.1
- net +5V: now also U4.3 (STBY), D6.1 (K), D7.1 (K); no longer C3.1, R4.1, U3.6 (Vout), U3.7 (Vout)
- new net 5V_BUCK: C3.1, D7.2 (A), R4.1, U3.6 (Vout), U3.7 (Vout)
- new net 5V_USB: D6.2 (A)
Other:
- moved on the sheet: C5, D3, R15
