File: PCB_Option_Maker/PCB_Module_Payement/untitled.kicad_sch (KiCad schematic)
At the start: 23 parts, among them J7 Conn_01x02, U1 FSV330AF, U3 171013801, U4 BU33SD5WG-TR, U5 FSV330AF

Commit message: update pcb
Parts:
- R10, R2: footprint Resistor_SMD:R_1206_3216Metric -> Resistor_SMD:R_0402_1005Metric
Changed lines of the file:
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@@
 			)
 		)
-		(property "Footprint" "Resistor_SMD:R_1206_3216Metric"
+		(property "Footprint" "Resistor_SMD:R_0402_1005Metric"
 			(at 105.41 111.76 0)
 			(effects
@@
 			)
 		)
-		(property "Footprint" "Resistor_SMD:R_1206_3216Metric"
+		(property "Footprint" "Resistor_SMD:R_0402_1005Metric"
 			(at 105.41 121.92 0)
 			(effects
