File: PCB_Option_Maker/PCB_Module_Payement/PCB_Module_Payement.kicad_pcb (KiCad board)
At the start: 4 copper layers, 45.1 x 61.1 mm, 68 parts, among them J1 Conn_02x07_Odd_Even, J3 Conn_01x08, J4 Conn_01x06, J5 Conn_01x08, J6 Conn_01x04, J7 Conn_01x02, J8 USB_C_Receptacle_USB2.0, J9 Conn_ST_STDC14, Q2 MMBT2222A, SW1 SW_Push, SW2 SW_Push, SW3 SW_Push, U1 FSV330AF, U2 STM32G431CBUx, U3 171013801, U4 BU33SD5WG-TR, U5 FSV330AF, U6 USBLC6-2SC6

Commit message: pcb update
Parts:
- C15: renamed from C19; moved to B.Cu
- C16: renamed from C3; moved to B.Cu
- C17: renamed from C1; moved to B.Cu
- C18: renamed from C2; moved to B.Cu
- D3, D4: moved to B.Cu
- J4: renamed from J9; moved to F.Cu
- J5: renamed from J7; moved to F.Cu
- J_Switch1: moved to F.Cu
- Q1: renamed from Q2; moved to B.Cu
- R12: renamed from R15; moved to B.Cu
- R13: renamed from R4; moved to B.Cu
- R14: renamed from R5; moved to B.Cu
- R15: renamed from R10; moved to B.Cu
- R16: renamed from R3; moved to B.Cu
- R17: renamed from R2; moved to B.Cu
- R18: renamed from R21; moved to B.Cu
- R19: renamed from R8; moved to B.Cu
- R5: renamed from R23; moved to F.Cu
- R6: renamed from R17; moved to F.Cu
- R7: renamed from R1; moved to F.Cu
- R8: renamed from R19; moved to F.Cu
- U3: renamed from U5; moved to F.Cu
- U5: renamed from U1; moved to F.Cu
- U6: renamed from U3; moved to B.Cu
- moved SW1 21.4 mm to (161.6, 88.4), turned to -90 degrees
- moved C16 18.4 mm to (169.8, 99.3)
- moved U5 17.0 mm to (172.3, 118.6), turned to -90 degrees
- moved R2 16.4 mm to (159.3, 94.2), turned to -90 degrees
- moved C8 16.1 mm to (160.4, 94.2), turned to 90 degrees
- moved R1 15.8 mm to (159.7, 95.8), turned to 180 degrees
- moved J_Switch1 14.9 mm to (180.1, 116.2), turned to 90 degrees
- moved C4 14.7 mm to (151.8, 105.5), turned to 180 degrees
- moved BZ1 11.8 mm to (145.1, 86.8), turned to 0 degrees
- moved R4 11.5 mm to (171.8, 104.8), turned to 0 degrees
- moved R12 10.6 mm to (170.1, 114.0), turned to -90 degrees
- moved R18 10.5 mm to (175.2, 114.0), turned to -90 degrees
- moved D1 10.2 mm to (172.3, 103.5), turned to 180 degrees
- moved U6 10.0 mm to (173.0, 103.7), turned to -90 degrees
- moved D3 9.45 mm to (171.6, 113.5), turned to -90 degrees
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- renumbered C17 to C1, C212 to C10, C14 to C11, C4 to C12, C6 to C13, C18 to C14, C13 to C2, C11 to C3, C211 to C4, C12 to C5, C5 to C6, C16 to C8, C10 to C9, D2 to D1, D5 to D2, D1 to D5, H4 to H3, H3 to H4, J6 to J1, J4 to J2, J8 to J6, J1 to J7, J5 to J8, L201 to L1, R9 to R1, R12 to R10, R7 to R2, R13 to R20, R6 to R3, R14 to R4, R20 to R9, U2 to U1, U4 to U2, U6 to U4
Connections:
- net /Modules/RXD renamed /Modules/Bt_RXD
- net /Modules/TXD renamed /Modules/Bt_TXD
- net /STM32/USB_DM renamed /STM32/USB_D-
- net /STM32/USB_DP renamed /STM32/USB_D+
- J2 pad 1: /Modules/KEY -> /Modules/STATE
- J2 pad 6: /Modules/STATE -> /Modules/KEY
- J3 pad 2: /Modules/SPI1_Miso -> /Modules/RSTO
- J3 pad 3: /Modules/SPI1_Mosi -> /Modules/SS
- J3 pad 4: /Modules/SS -> /Modules/SPI1_Mosi
- J3 pad 7: /Modules/IRQ -> /Modules/SPI1_Miso
- J3 pad 8: /Modules/RSTO -> /Modules/IRQ
- J7 pad 10: /STM32/PC15 -> /STM32/PF0
- J7 pad 11: /STM32/Pb1 -> /STM32/PA7
- J7 pad 12: /STM32/PA7 -> /STM32/Pb1
- J7 pad 3: /STM32/PF0 -> /STM32/PC13
- J7 pad 4: /STM32/PF1 -> /STM32/PC14
- J7 pad 6: /STM32/PC13 -> /STM32/PC15
- J7 pad 9: /STM32/PC14 -> /STM32/PF1
- U1 pad 25: /Modules/Culomn4 -> /Modules/R0W1
- U1 pad 26: /Modules/Culomn3 -> /Modules/ROW2
- U1 pad 27: /Modules/Culomn2 -> /Modules/ROW3
- U1 pad 28: /Modules/Culomn1 -> /Modules/ROW4
- U1 pad 29: /Modules/ROW4 -> /Modules/Culomn1
- U1 pad 30: /Modules/ROW3 -> /Modules/Culomn2
- U1 pad 31: /Modules/ROW2 -> /Modules/Culomn3
- U1 pad 32: /Modules/R0W1 -> /Modules/Culomn4
Routing:
- net GND: track 0.00 -> 54.1 mm, vias 0 -> 50
- net /STM32/PF0: track 0.00 -> 49.6 mm, vias 0 -> 1
- net /STM32/PF1: track 0.00 -> 47.2 mm, vias 0 -> 1
- net /STM32/PC14: track 0.00 -> 45.6 mm, vias 0 -> 1
- net /STM32/PC15: track 0.00 -> 45.5 mm, vias 0 -> 1
- net /STM32/PC13: track 0.00 -> 41.8 mm, vias 0 -> 1
- net /Modules/I2C1_SDA: track 0.00 -> 40.3 mm, vias 0 -> 1
- net /Modules/SPI1_SCK: track 0.00 -> 39.1 mm, vias 0 -> 2
- net /Modules/I2C1_SCL: track 0.00 -> 36.5 mm, vias 0 -> 1
- net /STM32/NRST: track 0.00 -> 35.3 mm, vias 0 -> 2
- net +3.3V: track 0.43 -> 33.9 mm, vias 0 -> 8
- net /STM32/BUZZER: track 0.00 -> 33.4 mm, vias 0 -> 1
- net /STM32/SWO: track 0.00 -> 29.4 mm, vias 0 -> 2
- net /Modules/STATE: track 0.00 -> 29.3 mm
- net /STM32/Pb1: track 0.00 -> 28.0 mm, vias 0 -> 1
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- added copper zone on In2.Cu, net +3.3V
- added copper zone on In2.Cu, net +5V
- added copper zone on In2.Cu, net VCC
Other:
- board size 45.1 x 61.1 mm -> 46.1 x 61.1 mm

Commit message: update pcb
Parts:
- R10: renamed from R15; footprint Resistor_SMD:R_1206_3216Metric -> Resistor_SMD:R_0402_1005Metric
- R2: renamed from R17; footprint Resistor_SMD:R_1206_3216Metric -> Resistor_SMD:R_0402_1005Metric
- renumbered C17 to C1, C9 to C10, C3 to C11, C5 to C12, C2 to C13, C11 to C14, C8 to C16, C1 to C17, C14 to C18, C15 to C19, C18 to C2, C4 to C211, C10 to C212, C16 to C3, C12 to C4, C6 to C5, C13 to C6, D5 to D1, D1 to D2, D2 to D5, H4 to H3, H3 to H4, J7 to J1, J2 to J4, J8 to J5, J1 to J6, J5 to J7, J6 to J8, J4 to J9, L1 to L201, Q1 to Q2, R7 to R1, R10 to R12, R20 to R13, R4 to R14, R12 to R15, R6 to R17, R8 to R19, R9 to R20, R18 to R21, R5 to R23, R16 to R3, R13 to R4, R14 to R5, R3 to R6, R2 to R7, R19 to R8, R1 to R9, U5 to U1, U1 to U2, U6 to U3, U2 to U4, U3 to U5, U4 to U6
Routing:
- net /Modules/I2C1_SDA: track 40.3 -> 32.9 mm
- net /STM32/SWDIO: track 21.0 -> 24.1 mm
- net /STM32/SWCLK: track 21.2 -> 24.2 mm
- net /Alim/Charge_Batterie: track 27.3 -> 29.5 mm
- net /STM32/SWO: track 29.4 -> 31.3 mm
- net /STM32/PC15: track 45.5 -> 44.1 mm
- net /STM32/PC14: track 45.6 -> 44.6 mm
- net /Modules/Culomn4: track 13.2 -> 14.2 mm
- net /STM32/PF1: track 47.2 -> 46.3 mm
- net GND: track 54.1 -> 55.1 mm, vias 50 -> 79
- net /STM32/PF0: track 49.6 -> 48.7 mm
- net VCC: track 8.04 -> 7.16 mm
- net /STM32/PC13: track 41.8 -> 41.0 mm
- net /Modules/SPI1_Miso: track 18.7 -> 19.3 mm
