File: PCB_Option_Maker/PCB_Module_Payement/PCB_Module_Payement.kicad_pcb (KiCad board)
At the start: 4 copper layers, 46.1 x 61.1 mm, 68 parts, among them J1 Conn_01x04, J2 Conn_01x06, J3 Conn_01x08, J4 Conn_ST_STDC14, J5 Conn_01x02, J6 USB_C_Receptacle_USB2.0, J7 Conn_02x07_Odd_Even, J8 Conn_01x08, Q1 MMBT2222A, SW1 SW_Push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

Commit message: stm32 test rfid
Parts:
- moved H1 0.07 mm to (139.1, 74.2)
- moved H2 0.07 mm to (178.7, 74.2)
- moved H4 0.07 mm to (178.7, 122.2)
Routing:
- net +3.3V: track 33.9 -> 36.5 mm, vias 8 -> 10
Changed lines of the file:
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@@
 	(footprint "MountingHole:MountingHole_2.7mm_M2.5_Pad"
 		(layer "F.Cu")
-		(at 178.7 122.2)
+		(at 178.65 122.15)
 		(descr "Mounting Hole 2.7mm, M2.5")
 		(tags "mounting hole 2.7mm m2.5")
@@
 	(footprint "MountingHole:MountingHole_2.7mm_M2.5_Pad"
 		(layer "F.Cu")
-		(at 139.05 122.15)
+		(at 139.1 122.15)
 		(descr "Mounting Hole 2.7mm, M2.5")
 		(tags "mounting hole 2.7mm m2.5")
@@
 	(footprint "MountingHole:MountingHole_2.7mm_M2.5_Pad"
 		(layer "F.Cu")
-		(at 178.7 74.15)
+		(at 178.65 74.2)
 		(descr "Mounting Hole 2.7mm, M2.5")
 		(tags "mounting hole 2.7mm m2.5")
 		(property "Reference" "H2"
-			(at 0 -3.7 0)
+			(at -3.65 -1.9 0)
 			(layer "F.SilkS")
 			(effects
@@
 	(footprint "MountingHole:MountingHole_2.7mm_M2.5_Pad"
 		(layer "F.Cu")
-		(at 139 74.15)
+		(at 139.05 74.2)
 		(descr "Mounting Hole 2.7mm, M2.5")
 		(tags "mounting hole 2.7mm m2.5")
 		(property "Reference" "H1"
-			(at 0 -3.7 0)
+			(at 0.35 4.2 0)
 			(layer "F.SilkS")
 			(effects
@@
 	)
 	(gr_line
-		(start 162.65 125.4)
+		(start 162.62 125.4)
 		(end 135.85 125.41)
 		(stroke
@@
 	)
 	(segment
+		(start 140.205 96.795)
+		(end 139.4 97.6)
+		(width 0.3)
+		(layer "F.Cu")
+		(net 7)
+	)
+	(segment
 		(start 165.65 99.56)
 		(end 164.65 99.56)
@@
 	)
 	(segment
+		(start 137.91 96.795)
+		(end 139.145 96.795)
+		(width 0.3)
+		(layer "F.Cu")
+		(net 7)
+	)
+	(segment
 		(start 156.15 106.4)
 		(end 156.5825 106.4)
@@
 	)
 	(segment
+		(start 139.145 96.795)
+		(end 139.15 96.8)
+		(width 0.3)
+		(layer "F.Cu")
+		(net 7)
+	)
+	(segment
 		(start 163.7 99.53)
 		(end 163.7 100.1)
@@
 	)
 	(segment
+		(start 140.45 96.795)
+		(end 140.205 96.795)
+		(width 0.3)
+		(layer "F.Cu")
+		(net 7)
+	)
+	(segment
 		(start 162.79 108.54)
 		(end 162.86 108.61)
@@
 	)
 	(via
+		(at 139.15 96.8)
+		(size 0.5)
+		(drill 0.3)
+		(layers "F.Cu" "B.Cu")
+		(net 7)
+	)
+	(via
 		(at 158.75 96.3)
 		(size 0.5)
@@
 		(net 7)
 	)
+	(via
+		(at 139.4 97.6)
+		(size 0.5)
+		(drill 0.3)
+		(layers "F.Cu" "B.Cu")
+		(net 7)
+	)
 	(segment
 		(start 154.09 102.91)
@@
 		(polygon
 			(pts
-				(xy 181.35 70.95) (xy 181.35 125.4) (xy 174.02 125.4) (xy 174.02 132.05) (xy 162.62 132.05) (xy 162.62 125.4)
+				(xy 181.95 70.95) (xy 181.9 125.4) (xy 174.02 125.4) (xy 174.02 132.05) (xy 162.62 132.05) (xy 162.62 125.4)
 				(xy 135.82 125.4) (xy 135.77 70.95)
 			)
@@
 		(polygon
 			(pts
-				(xy 181.35 70.95) (xy 181.35 125.4) (xy 174.02 125.4) (xy 174.02 132.05) (xy 162.62 132.05) (xy 162.62 125.4)
+				(xy 181.95 70.95) (xy 181.9 125.4) (xy 174.02 125.4) (xy 174.02 132.05) (xy 162.62 132.05) (xy 162.62 125.4)
 				(xy 135.82 125.4) (xy 135.77 70.95)
 			)
@@
 		(polygon
 			(pts
-				(xy 181.35 70.95) (xy 181.35 125.4) (xy 174.02 125.4) (xy 174.02 132.05) (xy 162.62 132.05) (xy 162.62 125.4)
+				(xy 181.95 70.95) (xy 181.9 125.4) (xy 174.02 125.4) (xy 174.02 132.05) (xy 162.62 132.05) (xy 162.62 125.4)
 				(xy 135.82 125.4) (xy 135.77 70.95)
 			)
@@
 		(polygon
 			(pts
-				(xy 162.62 125.4) (xy 162.62 132.05) (xy 174.02 132.05) (xy 174.02 125.4) (xy 181.35 125.4) (xy 181.35 70.95)
+				(xy 162.62 125.4) (xy 162.62 132.05) (xy 174.02 132.05) (xy 174.02 125.4) (xy 181.9 125.4) (xy 181.95 70.95)
 				(xy 135.77 70.95) (xy 135.77 88.6) (xy 162.65 88.55)
 			)
@@
 		(polygon
 			(pts
-				(xy 181.35 70.95) (xy 181.35 125.4) (xy 174.02 125.4) (xy 174.02 132.05) (xy 162.62 132.05) (xy 162.62 125.4)
+				(xy 181.95 70.95) (xy 181.9 125.4) (xy 174.02 125.4) (xy 174.02 132.05) (xy 162.62 132.05) (xy 162.62 125.4)
 				(xy 135.82 125.4) (xy 135.77 70.95)
 			)
